Commit message: Task1 - completed\n- Created expected robot model for visualization\n- Made final corrections to URDF specifications\n- Typo in pointing URDF file under launch file corrected

File: my_rb1_description/urdf/my_rb1_robot.urdf (robot description, URDF)
Before this commit: robot rb1_robot, 7 links, 6 joints
Links:
- link base_link: mass 18.5 -> 19
Joints:
- joint base_link_back_caster_joint: origin xyz=-0.1 0.0 -0.15 rpy=0 0 0 -> xyz=0.1 0.0 -0.15 rpy=0 0 0
- joint base_link_front_caster_joint: origin xyz=0.1 0.0 -0.15 rpy=0 0 0 -> xyz=-0.1 0.0 -0.15 rpy=0 0 0
